Commit message: fix submodule

File: src/scv_system/scv_tf/urdf/morai.urdf (robot description, URDF)
Before this commit: robot ssc, 3 links, 2 joints
Links:
- link base_link: geometry collision box size=0.9 0.45 0.5; visual box size=0.9 0.45 0.6
- link velodyne: mass 0.001 -> 0.925; geometry collision cylinder length=0.065 radius=0.0515; visual cylinder length=0.065 radius=0.0515
Joints:
- joint velodyne_joint: origin xyz=0 0 1 rpy=0 0 0 -> xyz=0 0 0.4325 rpy=0 0 0
