Commit message: submodule update

File: src/scv_system/scv_description/scv_tf/urdf/scv.urdf.xacro (robot description, xacro)
@@ -79,3 +79,18 @@
     <origin xyz="0.171 0 0.041" rpy="0 0 0"/>
   </joint>
+  <link name="cam">
+    <visual>
+      <geometry>
+        <box size="0.09 0.05 0.05"/>
+      </geometry>
+      <material name="blue">
+        <color rgba="0 0 0.9 1"/>
+      </material>
+    </visual>
+  </link>
+  <joint name="camera_joint" type="fixed">
+    <parent link="back_box"/>
+    <child link="cam"/>
+    <origin xyz="0.2 -0.17 0.125" rpy="0 0 -1.57"/>
+  </joint>
 </robot>

Commit message: update SCV

File: src/scv_system/scv_description/scv_tf/urdf/scv.urdf.xacro (robot description, xacro)
@@ -49,5 +49,5 @@
     <parent link="back_box"/>
     <child link="gps_antenna_link"/>
-    <origin xyz="0.1175 -0.1235 0.11" rpy="0 0 0"/>
+    <origin xyz="0.1175 0.0 0.11" rpy="0 0 0"/>
   </joint>
   <joint name="back_box_joint" type="fixed">
