Commit message: update system for SSC

File: src/vehicle/SSC/ssc_description/urdf/robot_main.urdf.xacro (robot description, xacro)
@@ -1,6 +1,6 @@
 <?xml version="1.0"?>
-<robot name="SSC_with_modular_sensors" xmlns:xacro="http://www.ros.org/wiki/xacro" xmlns:urdf="http://www.ros.org/wiki/urdf">
+<robot name="ssc_with_modular_sensors" xmlns:xacro="http://www.ros.org/wiki/xacro" xmlns:urdf="http://www.ros.org/wiki/urdf">
   <xacro:property name="M_PI" value="3.1415926535897931" />
-  <xacro:include filename="$(find SSC_description)/urdf/sensors/gps_sensor.urdf.xacro" />
+  <xacro:include filename="$(find ssc_description)/urdf/sensors/gps_sensor.urdf.xacro" />
   <xacro:include filename="$(find zed_wrapper)/urdf/zed_macro.urdf.xacro" />
   <!-- 차량의 주요 바디를 나타내는 base_link 정의 -->

File: src/vehicle/SSC/ssc_description/urdf/sensors/gps_sensor.urdf.xacro (robot description, xacro)
@@ -8,5 +8,5 @@
         <origin xyz="0 0 0" rpy="1.5708 0 0"/>
         <geometry>
-          <mesh filename="file://$(find SSC_description)/meshes/GNSS_antenna.stl" scale="0.0009 0.0009 0.0009"/>
+          <mesh filename="file://$(find ssc_description)/meshes/GNSS_antenna.stl" scale="0.0009 0.0009 0.0009"/>
         </geometry>
         <material name="white">

Commit message: update

File: src/vehicle/SSC/ssc_description/urdf/robot_main.urdf.xacro (robot description, xacro)
@@ -29,4 +29,9 @@
     <origin xyz="-0.2 0 0.6" rpy="0 0 0"/>
   </xacro:gps_sensor>
+  <joint name="d435i_to_chassis" type="fixed">
+    <parent link="chassis"/>
+    <child link="camera_link"/>
+    <origin xyz="0.2 0 0.45" rpy="0 0 0"/>
+  </joint>
   <xacro:zed_camera name="zed" model="zed2i" enable_gnss="true">
     <origin xyz="0 0 0" rpy="0 0 0"/>

Commit message: add d435i urdf

File: src/vehicle/SSC/ssc_description/urdf/robot_main.urdf.xacro (robot description, xacro)
@@ -4,4 +4,5 @@
   <xacro:include filename="$(find ssc_description)/urdf/sensors/gps_sensor.urdf.xacro" />
   <xacro:include filename="$(find zed_wrapper)/urdf/zed_macro.urdf.xacro" />
+  <xacro:include filename="$(find realsense2_description)/urdf/_d435i.urdf.xacro" />
   <!-- 차량의 주요 바디를 나타내는 base_link 정의 -->
   <link name="base_link">
@@ -29,9 +30,13 @@
     <origin xyz="-0.2 0 0.6" rpy="0 0 0"/>
   </xacro:gps_sensor>
-  <joint name="d435i_to_chassis" type="fixed">
+  <xacro:sensor_d435i name="camera_link" parent="chassis" use_nominal_extrinsics="true">
+    <origin xyz="0.7 0 0.08" rpy="0 0 0"/>
+  </xacro:sensor_d435i>
+<!--
+  <joint name="camera_to_chassis" type="fixed">
     <parent link="chassis"/>
     <child link="camera_link"/>
     <origin xyz="0.2 0 0.45" rpy="0 0 0"/>
-  </joint>
+  </joint> -->
   <xacro:zed_camera name="zed" model="zed2i" enable_gnss="true">
     <origin xyz="0 0 0" rpy="0 0 0"/>

Commit message: update mando contest

File: src/vehicle/SSC/ssc_description/urdf/robot_main.urdf.xacro (robot description, xacro)
@@ -42,8 +42,9 @@
     <origin xyz="0 0 0" rpy="0 0 0"/>
   </xacro:zed_camera>
+  <!--Camera Tilt-->
   <joint name="zed_to_chassis" type="fixed">
     <parent link="chassis"/>
     <child link="zed_camera_link"/>
-    <origin xyz="-0.2 0 0.45" rpy="0 0 0"/>
+    <origin xyz="-0.2 0 0.45" rpy="0 -0.1 0"/>
   </joint>
 </robot>
